File: ecu32.kicad_pcb (KiCad board)
At the start: 4 copper layers, 90 x 95 mm, 77 parts, among them J1 USB_B, J3 Conn_02x08_Counter_Clockwise, J4 Conn_02x08_Counter_Clockwise, J5 Conn_02x08_Counter_Clockwise, Q1 BC847BS, Q2 Si4800BDY, Q3 Si4800BDY, Q4 Si4800BDY, U1 ESP32-WROOM-32D, U10 LM358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

Commit message: fix error
Routing:
- net Net-(R17-Pad1): track 5.34 -> 6.61 mm
Changed lines of the file:
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@@
   (segment (start 120.6 64.3) (end 121.94 65.64) (width 0.4) (layer "F.Cu") (net 20))
   (segment (start 119.034 64.3) (end 120.6 64.3) (width 0.4) (layer "F.Cu") (net 20))
-  (segment (start 119.034 64.3) (end 119.194 64.14) (width 0.4) (layer "F.Cu") (net 20))
   (segment (start 119.034 65.57) (end 119.034 64.3) (width 0.4) (layer "F.Cu") (net 20))
   (segment (start 121.94 65.64) (end 131.25 65.64) (width 0.4) (layer "F.Cu") (net 20))
@@
   (segment (start 113.603 80.072) (end 114.428 80.072) (width 0.4) (layer "F.Cu") (net 33))
   (segment (start 115 76.15) (end 114.75 75.9) (width 0.4) (layer "F.Cu") (net 33))
+  (segment (start 113.603 78.802) (end 113.603 80.072) (width 0.4) (layer "F.Cu") (net 33))
   (segment (start 114.428 80.072) (end 115 79.5) (width 0.4) (layer "F.Cu") (net 33))
   (segment (start 114.641 72.559) (end 113.797 72.559) (width 0.4) (layer "F.Cu") (net 34))
@@
     (polygon
       (pts
-        (xy 117 86)
-        (xy 108.5 86.000327)
-        (xy 108.500989 94.400327)
-        (xy 117.250002 94.4)
+        (xy 117.000008 86.2)
+        (xy 108.500008 86.200327)
+        (xy 108.500937 93.000327)
+        (xy 117.24995 93)
         (xy 117.247714 106.255268)
         (xy 117.428006 117.737982)
@@
         (xy 118 118.8)
         (xy 118 117.25)
-        (xy 118 93.5)
-        (xy 109.75 93.5)
+        (xy 118 92.3)
+        (xy 109.75 92.3)
         (xy 109.75 87)
         (xy 118 87)

Commit message: commit
Parts:
- removed G***: LOGO, Graphics:argonavis40
Other:
- board text removed: "Engine controller"
- board text removed: "V1.3"
